File: Electrical Hardware/PCB 2nd version (Final Version)/Up/Up.sch (EAGLE design)
At the start: 44 parts

Commit message: EE
Parts:
- C_BAT, C_VA1, C_VCAP1, C_VCAP2: value 22uF -> 2.2uF
- C_V1, C_V2, C_V3, C_V4, C_VA2: value 22uF -> 0.1uF
- renumbered U$2 to CX5032GA
Changed lines of the file:
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@@
 <part name="GND2" library="SparkFun-PowerSymbols" deviceset="GND" device=""/>
 <part name="GND3" library="SparkFun-PowerSymbols" deviceset="GND" device=""/>
-<part name="C_V3" library="SparkFun-Capacitors" deviceset="22UF" device="-0805-6.3V-20%" value="22uF"/>
-<part name="C_BAT" library="SparkFun-Capacitors" deviceset="22UF" device="-0805-6.3V-20%" value="22uF"/>
-<part name="C_VA1" library="SparkFun-Capacitors" deviceset="22UF" device="-0805-6.3V-20%" value="22uF"/>
-<part name="C_VA2" library="SparkFun-Capacitors" deviceset="22UF" device="-0805-6.3V-20%" value="22uF"/>
-<part name="C_V1" library="SparkFun-Capacitors" deviceset="22UF" device="-0805-6.3V-20%" value="22uF"/>
+<part name="C_V3" library="SparkFun-Capacitors" deviceset="22UF" device="-0805-6.3V-20%" value="0.1uF"/>
+<part name="C_BAT" library="SparkFun-Capacitors" deviceset="22UF" device="-0805-6.3V-20%" value="2.2uF"/>
+<part name="C_VA1" library="SparkFun-Capacitors" deviceset="22UF" device="-0805-6.3V-20%" value="2.2uF"/>
+<part name="C_VA2" library="SparkFun-Capacitors" deviceset="22UF" device="-0805-6.3V-20%" value="0.1uF"/>
+<part name="C_V1" library="SparkFun-Capacitors" deviceset="22UF" device="-0805-6.3V-20%" value="0.1uF"/>
 <part name="GND4" library="SparkFun-PowerSymbols" deviceset="GND" device=""/>
-<part name="C_V4" library="SparkFun-Capacitors" deviceset="22UF" device="-0805-6.3V-20%" value="22uF"/>
-<part name="C_VCAP1" library="SparkFun-Capacitors" deviceset="22UF" device="-0805-6.3V-20%" value="22uF"/>
+<part name="C_V4" library="SparkFun-Capacitors" deviceset="22UF" device="-0805-6.3V-20%" value="0.1uF"/>
+<part name="C_VCAP1" library="SparkFun-Capacitors" deviceset="22UF" device="-0805-6.3V-20%" value="2.2uF"/>
 <part name="GND6" library="SparkFun-PowerSymbols" deviceset="GND" device=""/>
-<part name="C_V2" library="SparkFun-Capacitors" deviceset="22UF" device="-0805-6.3V-20%" value="22uF"/>
-<part name="C_VCAP2" library="SparkFun-Capacitors" deviceset="22UF" device="-0805-6.3V-20%" value="22uF"/>
+<part name="C_V2" library="SparkFun-Capacitors" deviceset="22UF" device="-0805-6.3V-20%" value="0.1uF"/>
+<part name="C_VCAP2" library="SparkFun-Capacitors" deviceset="22UF" device="-0805-6.3V-20%" value="2.2uF"/>
 <part name="GND5" library="SparkFun-PowerSymbols" deviceset="GND" device=""/>
 <part name="GND19" library="SparkFun-PowerSymbols" deviceset="GND" device=""/>
@@
 <part name="C2" library="SparkFun-Capacitors" deviceset="22PF" device="-0603-50V-5%" value="12pF"/>
 <part name="GND22" library="SparkFun-Aesthetics" deviceset="GND" device=""/>
-<part name="U$2" library="Cristal Oscillator" deviceset="OSC" device=""/>
+<part name="CX5032GA" library="Cristal Oscillator" deviceset="OSC" device=""/>
 <part name="LM" library="headers(2mm)" deviceset="1X4" device=""/>
 <part name="RM" library="headers(2mm)" deviceset="1X4" device=""/>
@@
 <instance part="C2" gate="G$1" x="24.08" y="82.9"/>
 <instance part="GND22" gate="1" x="24.08" y="67.66"/>
-<instance part="U$2" gate="G$1" x="39.32" y="98.521"/>
+<instance part="CX5032GA" gate="G$1" x="39.32" y="98.521"/>
 <instance part="LM" gate="G$1" x="270.46" y="24.48" rot="R90"/>
 <instance part="RM" gate="G$1" x="290.78" y="24.48" rot="R90"/>
@@
 <wire x1="54.56" y1="105.76" x2="54.56" y2="98.14" width="0.1524" layer="91"/>
 <label x="54.56" y="105.76" size="0.8128" layer="95" rot="R90" xref="yes"/>
-<pinref part="U$2" gate="G$1" pin="IN2"/>
+<pinref part="CX5032GA" gate="G$1" pin="IN2"/>
 <wire x1="54.56" y1="98.14" x2="54.56" y2="87.98" width="0.1524" layer="91"/>
 <wire x1="51.06" y1="98.141" x2="51.06" y2="98.14" width="0.1524" layer="91"/>
@@
 <wire x1="24.08" y1="105.76" x2="24.08" y2="98.14" width="0.1524" layer="91"/>
 <label x="24.08" y="105.76" size="0.8128" layer="95" rot="R90" xref="yes"/>
-<pinref part="U$2" gate="G$1" pin="IN1"/>
+<pinref part="CX5032GA" gate="G$1" pin="IN1"/>
 <wire x1="24.08" y1="98.14" x2="24.08" y2="87.98" width="0.1524" layer="91"/>
 <wire x1="27.36" y1="98.141" x2="27.36" y2="98.14" width="0.1524" layer="91"/>

Commit message: 3week Meeting
Parts:
- renumbered CX5032GA to CX5032GA*8MHZ*CYSTAL
Changed lines of the file:
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@@
 <?xml version="1.0" encoding="utf-8"?>
 <!DOCTYPE eagle SYSTEM "eagle.dtd">
-<eagle version="8.6.0">
+<eagle version="8.2.2">
 <drawing>
 <settings>
@@
 <part name="C2" library="SparkFun-Capacitors" deviceset="22PF" device="-0603-50V-5%" value="12pF"/>
 <part name="GND22" library="SparkFun-Aesthetics" deviceset="GND" device=""/>
-<part name="CX5032GA" library="Cristal Oscillator" deviceset="OSC" device=""/>
+<part name="CX5032GA*8MHZ*CYSTAL" library="Cristal Oscillator" deviceset="OSC" device=""/>
 <part name="LM" library="headers(2mm)" deviceset="1X4" device=""/>
 <part name="RM" library="headers(2mm)" deviceset="1X4" device=""/>
@@
 <part name="U$7" library="adafruit" library_urn="urn:adsk.eagle:library:420" deviceset="PINHD-1X10" device=""/>
 <part name="GND13" library="SparkFun-Aesthetics" deviceset="GND" device=""/>
-<part name="JP1" library="pinhead" library_urn="urn:adsk.eagle:library:325" deviceset="PINHD-1X2" device="" package3d_urn="urn:adsk.eagle:package:22435/2"/>
-<part name="JP2" library="pinhead" library_urn="urn:adsk.eagle:library:325" deviceset="PINHD-1X4" device="" package3d_urn="urn:adsk.eagle:package:22407/2"/>
+<part name="JP1" library="pinhead" library_urn="urn:adsk.eagle:library:325" deviceset="PINHD-1X2" device=""/>
+<part name="JP2" library="pinhead" library_urn="urn:adsk.eagle:library:325" deviceset="PINHD-1X4" device=""/>
 <part name="U$8" library="headers(2mm)" deviceset="1X4" device=""/>
 <part name="RSTR" library="SparkFun-Resistors" deviceset="0.75OHM" device="-0805-1/4W-1%" value="10K"/>
@@
 <instance part="C2" gate="G$1" x="24.08" y="82.9"/>
 <instance part="GND22" gate="1" x="24.08" y="67.66"/>
-<instance part="CX5032GA" gate="G$1" x="39.32" y="98.521"/>
+<instance part="CX5032GA*8MHZ*CYSTAL" gate="G$1" x="39.32" y="98.521"/>
 <instance part="LM" gate="G$1" x="270.46" y="24.48" rot="R90"/>
 <instance part="RM" gate="G$1" x="290.78" y="24.48" rot="R90"/>
@@
 <wire x1="54.56" y1="105.76" x2="54.56" y2="98.14" width="0.1524" layer="91"/>
 <label x="54.56" y="105.76" size="0.8128" layer="95" rot="R90" xref="yes"/>
-<pinref part="CX5032GA" gate="G$1" pin="IN2"/>
+<pinref part="CX5032GA*8MHZ*CYSTAL" gate="G$1" pin="IN2"/>
 <wire x1="54.56" y1="98.14" x2="54.56" y2="87.98" width="0.1524" layer="91"/>
 <wire x1="51.06" y1="98.141" x2="51.06" y2="98.14" width="0.1524" layer="91"/>
@@
 <wire x1="24.08" y1="105.76" x2="24.08" y2="98.14" width="0.1524" layer="91"/>
 <label x="24.08" y="105.76" size="0.8128" layer="95" rot="R90" xref="yes"/>
-<pinref part="CX5032GA" gate="G$1" pin="IN1"/>
+<pinref part="CX5032GA*8MHZ*CYSTAL" gate="G$1" pin="IN1"/>
 <wire x1="24.08" y1="98.14" x2="24.08" y2="87.98" width="0.1524" layer="91"/>
 <wire x1="27.36" y1="98.141" x2="27.36" y2="98.14" width="0.1524" layer="91"/>
@@
 <compatibility>
 <note version="8.2" severity="warning">
-Since Version 8.2, EAGLE supports online libraries. The ids
+Since Version 8.2, Eagle supports online libraries. The ids
 of those online libraries will not be understood (or retained)
 with this version.
 </note>
-<note version="8.3" severity="warning">
-Since Version 8.3, EAGLE supports URNs for individual library
-assets (packages, symbols, and devices). The URNs of those assets
-will not be understood (or retained) with this version.
-</note>
-<note version="8.3" severity="warning">
-Since Version 8.3, EAGLE supports the association of 3D packages
-with devices in libraries, schematics, and board files. Those 3D
-packages will not be understood (or retained) with this version.
-</note>
 </compatibility>
