File: Electrical Hardware/PCB 2nd version/Down/Down.sch (EAGLE design)
At the start: 88 parts

Commit message: PCB 3rd version
Changed lines of the file:
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@@
+</nets>
+</sheet>
+<sheet>
+<plain>
+</plain>
+<instances>
+</instances>
+<busses>
+</busses>
+<nets>
 </nets>
 </sheet>
