File: Electrical Hardware/PCB 3rd version (Final Version)/Peripherals.brd (EAGLE design)
At the start: 100 x 80 mm, 89 parts

Commit message: PCB 3rd version
Parts:
- removed LED2, LED3: BLUE, SparkFun-LED:LED-1206
- removed LED_R2, LED_R3: 1k, SparkFun-Resistors:0805
- removed P2, P3: (no value), jst-ph:JST-PH2
- added CEM10, CEM9: 0.1µF, SparkFun-Capacitors:0805
- added U$2, U$3: 1X1, headers(2mm):1X1
- added U$8, U$9: 1X2, headers(2mm):1X2
- moved R_EM5 377.9 mm to (72.0, 77.0), turned to 270 degrees
- moved R_EM1 373.5 mm to (68.0, 77.0), turned to 90 degrees
- moved R_EM7 371.7 mm to (82.0, 76.0), turned to 90 degrees
- moved R_EM3 369.1 mm to (86.0, 76.0), turned to 90 degrees
- moved CEM4 360.4 mm to (100.0, 68.0)
- moved CEM3 359.3 mm to (101.0, 66.0), turned to 180 degrees
- moved R_EM4 359.1 mm to (48.0, 47.0), turned to 270 degrees
- moved RRE3 358.5 mm to (99.0, 70.0), turned to 180 degrees
- moved CEM2 357.9 mm to (55.0, 70.0), turned to 180 degrees
- moved RRE2 355.1 mm to (54.0, 68.0)
- moved R_EM 354.2 mm to (53.0, 66.0)
- moved U$1 349.0 mm to (93.0, 62.0), turned to 180 degrees
- moved CEM1 348.9 mm to (51.0, 61.0)
- moved R_EM2 348.3 mm to (103.0, 61.0), turned to 180 degrees
- moved RRE4 347.7 mm to (104.0, 59.0), turned to 180 degrees
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Connections:
- removed net LED1: LED_R1.2, LED_R2.2, LED_R3.2
- removed net N$10: LED3.A, LED_R3.1
- removed net N$9: LED2.A, LED_R2.1
- net 3.3V: now also LED_R1.2, U$2.1
- net A5V: now also CEM10.1, CEM9.1
- net AGND: now also CEM10.2, CEM9.2
- net EM_L: now also U$8.1; no longer P2.1
- net EM_R: now also U$9.2; no longer P3.1
- net GND: now also U$3.1; no longer LED2.C, LED3.C
- net RE_L: now also U$8.2; no longer P2.2
- net RE_R: now also U$9.1; no longer P3.2
- net RE_RFA: now also RE_RFB.E, RRE4.2; no longer RE_RFA.E, RRE3.2
- net RE_RFB: now also RE_RFA.E, RRE3.2; no longer RE_RFB.E, RRE4.2
Routing:
- added copper zone on layer 1, net A5V
- added copper zone on layer 16, net AGND
Other:
- board size 100 x 80 mm -> 82 x 37 mm

Commit message: PCB 3rd v upd
Parts:
- removed MGND: 0, SparkFun-Resistors:0805
- moved CC5 366.7 mm to (207.0, 17.0), turned to 180 degrees
- moved CC6 362.2 mm to (203.0, 17.0), turned to 180 degrees
- moved CC4 358.4 mm to (-11.0, 2.00), turned to 180 degrees
- moved CC7 358.0 mm to (199.0, 17.0), turned to 180 degrees
- moved CC8 353.8 mm to (195.0, 17.0), turned to 180 degrees
- moved CC3 353.3 mm to (-7.00, 2.00), turned to 180 degrees
- moved CC2 348.3 mm to (-3.00, 2.00), turned to 180 degrees
- moved CC1 343.4 mm to (1.00, 2.00), turned to 180 degrees
- moved CC 338.6 mm to (5.00, 2.00), turned to 180 degrees
- moved CB2 334.0 mm to (9.00, 2.00), turned to 180 degrees
- moved CB1 329.5 mm to (13.0, 2.00), turned to 180 degrees
- moved U$18 325.5 mm to (88.0, 48.0), turned to 270 degrees
- moved AGND 325.1 mm to (17.0, 2.00), turned to 180 degrees
- moved U$16 324.0 mm to (66.0, 48.0), turned to 90 degrees
- moved GND 323.0 mm to (159.0, 17.0), turned to 180 degrees
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Connections:
- net BGND: no longer AGND.1, GND.1, MGND.1
- net MGND: now also AGND.1, GND.1; no longer MGND.2

Commit message: ..........
Parts:
- added R_VMTR_1: 10K, SparkFun-Resistors:0805
- added R_VMTR_2: 20K, SparkFun-Resistors:0805
- added U$11, U$12: 1X1, headers(2mm):1X1
- moved REG1 99.3 mm to (67.0, 58.0), turned to 90 degrees
- moved RM 97.7 mm to (92.0, 46.0)
- moved CB2 80.1 mm to (79.0, 41.0), turned to 0 degrees
- moved REG2 75.7 mm to (87.0, 58.0), turned to 90 degrees
- moved CB1 73.2 mm to (75.0, 41.0)
- moved U$2 72.4 mm to (95.0, 59.0)
- moved REG3 71.6 mm to (77.0, 52.0), turned to 90 degrees
- moved R_LMC_1 67.1 mm to (33.0, 61.0)
- moved LM 63.1 mm to (62.0, 46.0)
- moved U$3 60.2 mm to (95.0, 57.0)
- moved R_LMC_2 60.0 mm to (37.0, 57.0)
- moved U$15 47.5 mm to (52.0, 41.0), turned to 270 degrees
- moved R_RMC_1 37.5 mm to (98.0, 30.0)
- moved R_RMC_2 37.5 mm to (94.0, 30.0)
- moved U$17 28.8 mm to (102.0, 41.0), turned to 270 degrees
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Connections:
- removed net BGND: BAT.2, CB1.2, CB2.2
- new net VMTR: R_VMTR_1.2, R_VMTR_2.1, U$11.1
- net AGND: now also R_VMTR_1.1, U$12.1
- net MGND: now also BAT.2, CB1.2, CB2.2
- net VBAT: now also R_VMTR_2.2
Routing:
- net OUT_B: track 0.00 -> 15.4 mm
- net L: track 0.00 -> 11.6 mm, vias 0 -> 1
- net N$28: track 0.00 -> 9.10 mm, vias 0 -> 1
- net OUT_A: track 0.00 -> 3.98 mm
- net AGND: track 0.00 -> 3.58 mm, vias 0 -> 2
- net MGND: track 0.00 -> 2.24 mm, vias 0 -> 2
- net RE_L: track 0.00 -> 1.81 mm
- added copper zone on layer 16, net GND
- added copper zone on layer 16, net MGND
- added copper zone on layer 1, net VBAT

Commit message: Finshing PCB 3rd version Peripheral Board
Parts:
- added AGND1: 0, SparkFun-Resistors:0805
- added LED2: BLUE, SparkFun-LED:LED-1206
- added LED_R2: 1k, SparkFun-Resistors:0805
- moved R_VMTR_2 245.9 mm to (62.0, 55.0), turned to 270 degrees
- moved R_VMTR_1 245.0 mm to (61.0, 59.0), turned to 270 degrees
- moved CC5 141.7 mm to (73.0, 63.0), turned to 0 degrees
- moved CC7 131.5 mm to (72.0, 51.0), turned to 90 degrees
- moved CC6 119.5 mm to (90.0, 56.0), turned to 270 degrees
- moved CC8 118.0 mm to (82.0, 51.0), turned to 270 degrees
- moved CC3 101.5 mm to (79.0, 56.0), turned to 90 degrees
- moved CC4 101.5 mm to (75.0, 56.0), turned to 270 degrees
- moved CC1 101.0 mm to (87.0, 55.0), turned to 0 degrees
- moved CC 89.1 mm to (68.0, 65.0)
- moved CC2 86.1 mm to (64.0, 56.0), turned to 90 degrees
- moved CRMC_1 85.0 mm to (104.0, 42.0)
- moved CPWR_9 82.3 mm to (86.0, 65.0), turned to 0 degrees
- moved LED_R1 81.0 mm to (72.0, 68.0)
- moved GND 78.3 mm to (88.0, 50.0), turned to 90 degrees
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Connections:
- removed net N$28: LEFTMOTOR.2, U$16.N2D/P2D
- new net N$10: LED2.A, LED_R2.1
- new net N$9: LEFTMOTOR.1, U$16.N2D/P2D
- net 3.3V: no longer LED_R1.2
- net A5V: now also LED_R1.2, LED_R2.2
- net AGND: now also AGND1.2, LED1.C, LED2.C
- net GND: no longer LED1.C
- net L: now also LEFTMOTOR.2; no longer LEFTMOTOR.1
- net LPWMA: now also LM.3; no longer LM.4
- net LPWMB: now also LM.4; no longer LM.3
- net MGND: now also AGND1.1
- net OUTA: now also U$17.OUT_B; no longer U$17.OUT_A
- net OUTB: now also U$17.OUT_A; no longer U$17.OUT_B
- net RPWMA: now also RM.2; no longer RM.1
- net RPWMB: now also RM.1; no longer RM.2
Routing:
- net AGND: track 3.58 -> 59.6 mm, vias 2 -> 33
- net GND: track 0.00 -> 48.7 mm, vias 0 -> 12
- net 5V: track 0.00 -> 44.0 mm, vias 0 -> 6
- net VBAT: track 0.00 -> 41.6 mm
- net MGND: track 2.24 -> 37.0 mm, vias 2 -> 18
- net RE_R: track 0.00 -> 27.2 mm, vias 0 -> 2
- net RE_L: track 1.81 -> 26.9 mm, vias 0 -> 3
- net 3.3V: track 0.00 -> 16.8 mm
- net EM_L: track 0.00 -> 15.8 mm, vias 0 -> 2
- net EM_R: track 0.00 -> 14.9 mm, vias 0 -> 2
- net RE_LFA: track 0.00 -> 14.4 mm
- net RE_RFA: track 0.00 -> 12.7 mm
- net EM_LF: track 0.00 -> 11.6 mm
- net RENCA: track 0.00 -> 11.5 mm
- net N$9: track 0.00 -> 11.3 mm, vias 0 -> 1
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- added copper zone on layer 1, net 5V
Other:
- outline, holes or cut-outs redrawn
- board text added: "1st"
- board text added: "Eins"
- board text added: "The"
- board text added: "Triton"
- board text added: "UCSD"
- board text added: "~~~"
