File: Electrical Hardware/PCB 3rd version (Final Version)/Peripherals.sch (EAGLE design)
At the start: 89 parts

Commit message: PCB 3rd v upd
Parts:
- removed MGND: 0, SparkFun-Resistors:0.75OHM-0805-1/4W-1%
Connections:
- net BGND: no longer AGND.1, GND.1, MGND.1
- net MGND: now also AGND.1, GND.1; no longer MGND.2
Changed lines of the file:
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@@
 <?xml version="1.0" encoding="utf-8"?>
 <!DOCTYPE eagle SYSTEM "eagle.dtd">
-<eagle version="8.6.0">
+<eagle version="9.0.0">
 <drawing>
 <settings>
@@
 <part name="U$10" library="headers(2mm)" deviceset="1X3" device=""/>
 <part name="U$1" library="headers(2mm)" deviceset="1X3" device=""/>
-<part name="MGND" library="SparkFun-Resistors" library_urn="urn:adsk.eagle:library:532" deviceset="0.75OHM" device="-0805-1/4W-1%" value="0"/>
 <part name="AGND" library="SparkFun-Resistors" library_urn="urn:adsk.eagle:library:532" deviceset="0.75OHM" device="-0805-1/4W-1%" value="0"/>
 <part name="GND" library="SparkFun-Resistors" library_urn="urn:adsk.eagle:library:532" deviceset="0.75OHM" device="-0805-1/4W-1%" value="0"/>
@@
 <instance part="U$10" gate="G$1" x="-266.7" y="20.32"/>
 <instance part="U$1" gate="G$1" x="-93.98" y="22.86"/>
-<instance part="MGND" gate="G$1" x="25.4" y="-43.18" rot="R90"/>
 <instance part="AGND" gate="G$1" x="38.1" y="-40.64" rot="R90"/>
 <instance part="GND" gate="G$1" x="50.8" y="-43.18" rot="R90"/>
@@
 </segment>
 <segment>
-<pinref part="MGND" gate="G$1" pin="2"/>
-<wire x1="25.4" y1="-38.1" x2="25.4" y2="-33.02" width="0.1524" layer="91"/>
 <label x="25.4" y="-33.02" size="1.778" layer="95" rot="R90" xref="yes"/>
+<pinref part="AGND" gate="G$1" pin="1"/>
+<pinref part="GND" gate="G$1" pin="1"/>
+<wire x1="38.1" y1="-45.72" x2="38.1" y2="-48.26" width="0.1524" layer="91"/>
+<wire x1="38.1" y1="-48.26" x2="38.1" y2="-55.88" width="0.1524" layer="91"/>
+<wire x1="25.4" y1="-48.26" x2="38.1" y2="-48.26" width="0.1524" layer="91"/>
+<junction x="38.1" y="-48.26"/>
+<wire x1="38.1" y1="-48.26" x2="50.8" y2="-48.26" width="0.1524" layer="91"/>
+<label x="38.1" y="-55.88" size="1.778" layer="95" rot="R270" xref="yes"/>
+<wire x1="25.4" y1="-33.02" x2="25.4" y2="-48.26" width="0.1524" layer="91"/>
 </segment>
 </net>
@@
 <net name="BGND" class="0">
 <segment>
-<pinref part="MGND" gate="G$1" pin="1"/>
-<pinref part="AGND" gate="G$1" pin="1"/>
-<pinref part="GND" gate="G$1" pin="1"/>
-<wire x1="38.1" y1="-45.72" x2="38.1" y2="-48.26" width="0.1524" layer="91"/>
-<wire x1="38.1" y1="-48.26" x2="38.1" y2="-55.88" width="0.1524" layer="91"/>
-<wire x1="25.4" y1="-48.26" x2="38.1" y2="-48.26" width="0.1524" layer="91"/>
-<junction x="38.1" y="-48.26"/>
-<wire x1="38.1" y1="-48.26" x2="50.8" y2="-48.26" width="0.1524" layer="91"/>
-<label x="38.1" y="-55.88" size="1.778" layer="95" rot="R270" xref="yes"/>
-</segment>
-<segment>
 <pinref part="BAT" gate="G$1" pin="2"/>

Commit message: ..........
Parts:
- added R_VMTR_1: 10K, SparkFun-Resistors:0.75OHM-0805-1/4W-1%
- added R_VMTR_2: 20K, SparkFun-Resistors:0.75OHM-0805-1/4W-1%
- added U$11, U$12: 1X1, headers(2mm):1X1
Connections:
- removed net BGND: BAT.2, CB1.2, CB2.2
- new net VMTR: R_VMTR_1.2, R_VMTR_2.1, U$11.1
- net AGND: now also R_VMTR_1.1, U$12.1
- net MGND: now also BAT.2, CB1.2, CB2.2
- net VBAT: now also R_VMTR_2.2
Changed lines of the file:
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@@
 <part name="U$8" library="headers(2mm)" deviceset="1X2" device=""/>
 <part name="U$9" library="headers(2mm)" deviceset="1X2" device=""/>
+<part name="R_VMTR_1" library="SparkFun-Resistors" deviceset="0.75OHM" device="-0805-1/4W-1%" value="10K"/>
+<part name="R_VMTR_2" library="SparkFun-Resistors" deviceset="0.75OHM" device="-0805-1/4W-1%" value="20K"/>
+<part name="U$11" library="headers(2mm)" deviceset="1X1" device=""/>
+<part name="U$12" library="headers(2mm)" deviceset="1X1" device=""/>
 </parts>
 <sheets>
@@
 <instance part="U$8" gate="G$1" x="-279.4" y="-127"/>
 <instance part="U$9" gate="G$1" x="-119.38" y="-124.46"/>
+<instance part="R_VMTR_1" gate="G$1" x="96.52" y="-48.26" rot="R90"/>
+<instance part="R_VMTR_2" gate="G$1" x="96.52" y="-30.48" rot="R90"/>
+<instance part="U$11" gate="G$1" x="111.76" y="-45.72" rot="R90"/>
+<instance part="U$12" gate="G$1" x="147.32" y="-20.32"/>
 </instances>
 <busses>
@@
 <junction x="195.58" y="-81.28"/>
 </segment>
+<segment>
+<pinref part="R_VMTR_2" gate="G$1" pin="2"/>
+<wire x1="96.52" y1="-25.4" x2="96.52" y2="-22.86" width="0.1524" layer="91"/>
+<label x="96.52" y="-22.86" size="1.016" layer="95" rot="R90" xref="yes"/>
+</segment>
 </net>
 <net name="LENCA" class="0">
@@
 </segment>
 <segment>
-<label x="25.4" y="-33.02" size="1.778" layer="95" rot="R90" xref="yes"/>
 <pinref part="AGND" gate="G$1" pin="1"/>
 <pinref part="GND" gate="G$1" pin="1"/>
 <wire x1="38.1" y1="-45.72" x2="38.1" y2="-48.26" width="0.1524" layer="91"/>
 <wire x1="38.1" y1="-48.26" x2="38.1" y2="-55.88" width="0.1524" layer="91"/>
-<wire x1="25.4" y1="-48.26" x2="38.1" y2="-48.26" width="0.1524" layer="91"/>
 <junction x="38.1" y="-48.26"/>
 <wire x1="38.1" y1="-48.26" x2="50.8" y2="-48.26" width="0.1524" layer="91"/>
 <label x="38.1" y="-55.88" size="1.778" layer="95" rot="R270" xref="yes"/>
-<wire x1="25.4" y1="-33.02" x2="25.4" y2="-48.26" width="0.1524" layer="91"/>
+</segment>
+<segment>
+<pinref part="BAT" gate="G$1" pin="2"/>
+<wire x1="68.58" y1="-53.34" x2="71.12" y2="-50.8" width="0.1524" layer="91"/>
+<label x="76.2" y="-45.72" size="0.8128" layer="95" rot="R90" xref="yes"/>
+<pinref part="CB1" gate="G$1" pin="2"/>
+<wire x1="71.12" y1="-50.8" x2="76.2" y2="-45.72" width="0.1524" layer="91"/>
+<wire x1="71.12" y1="-48.26" x2="71.12" y2="-50.8" width="0.1524" layer="91"/>
+<junction x="71.12" y="-50.8"/>
+<pinref part="CB2" gate="G$1" pin="2"/>
+<wire x1="71.12" y1="-48.26" x2="71.12" y2="-35.56" width="0.1524" layer="91"/>
+<junction x="71.12" y="-48.26"/>
 </segment>
 </net>
@@
 <label x="38.1" y="-33.02" size="1.778" layer="95" rot="R90" xref="yes"/>
 </segment>
+<segment>
+<pinref part="R_VMTR_1" gate="G$1" pin="1"/>
+<wire x1="96.52" y1="-53.34" x2="96.52" y2="-55.88" width="0.1524" layer="91"/>
+<label x="96.52" y="-55.88" size="1.778" layer="95" rot="R270" xref="yes"/>
+</segment>
+<segment>
+<pinref part="U$12" gate="G$1" pin="1"/>
+<wire x1="149.86" y1="-20.32" x2="152.4" y2="-20.32" width="0.1524" layer="91"/>
+<label x="152.4" y="-20.32" size="0.8128" layer="95" xref="yes"/>
+</segment>
 </net>
 <net name="A5V" class="0">
@@
 </segment>
 </net>
-<net name="BGND" class="0">
-<segment>
-<pinref part="BAT" gate="G$1" pin="2"/>
-<wire x1="68.58" y1="-53.34" x2="71.12" y2="-50.8" width="0.1524" layer="91"/>
-<label x="76.2" y="-45.72" size="0.8128" layer="95" rot="R90" xref="yes"/>
-<pinref part="CB1" gate="G$1" pin="2"/>
-<wire x1="71.12" y1="-50.8" x2="76.2" y2="-45.72" width="0.1524" layer="91"/>
-<wire x1="71.12" y1="-48.26" x2="71.12" y2="-50.8" width="0.1524" layer="91"/>
-<junction x="71.12" y="-50.8"/>
-<pinref part="CB2" gate="G$1" pin="2"/>
-<wire x1="71.12" y1="-48.26" x2="71.12" y2="-35.56" width="0.1524" layer="91"/>
-<junction x="71.12" y="-48.26"/>
-</segment>
-</net>
 <net name="N$8" class="0">
 <segment>
@@
 </segment>
 </net>
+<net name="VMTR" class="0">
+<segment>
+<pinref part="R_VMTR_2" gate="G$1" pin="1"/>
+<pinref part="R_VMTR_1" gate="G$1" pin="2"/>
+<label x="96.52" y="-40.64" size="1.016" layer="95" xref="yes"/>
+<wire x1="96.52" y1="-35.56" x2="96.52" y2="-40.64" width="0.1524" layer="91"/>
+<pinref part="U$11" gate="G$1" pin="1"/>
+<wire x1="96.52" y1="-40.64" x2="96.52" y2="-43.18" width="0.1524" layer="91"/>
+<wire x1="96.52" y1="-40.64" x2="111.76" y2="-40.64" width="0.1524" layer="91"/>
+<wire x1="111.76" y1="-40.64" x2="111.76" y2="-43.18" width="0.1524" layer="91"/>
+<junction x="96.52" y="-40.64"/>
+</segment>
+</net>
