File: Electrical Hardware/PCB 3rd version (Final Version)/peripheral/Peripherals.sch (EAGLE design)
At the start: 89 parts

Commit message: update PCB 3rd v
Parts:
- removed MGND: 0, SparkFun-Resistors:0.75OHM-0805-1/4W-1%
- added AGND1: 0, SparkFun-Resistors:0.75OHM-0805-1/4W-1%
- added LED2: BLUE, SparkFun-LED:LED-BLUE1206
- added LED_R2: 1k, SparkFun-Resistors:0.75OHM-0805-1/4W-1%
- added R_VMTR_1: 10K, SparkFun-Resistors:0.75OHM-0805-1/4W-1%
- added R_VMTR_2: 20K, SparkFun-Resistors:0.75OHM-0805-1/4W-1%
- added U$11, U$12: 1X1, headers(2mm):1X1
Connections:
- removed net BGND: AGND.1, BAT.2, CB1.2, CB2.2, GND.1, MGND.1
- removed net N$28: LEFTMOTOR.2, U$16.N2D/P2D
- new net N$10: LED2.A, LED_R2.1
- new net N$9: LEFTMOTOR.1, U$16.N2D/P2D
- new net VMTR: R_VMTR_1.2, R_VMTR_2.1, U$11.1
- net 3.3V: no longer LED_R1.2
- net A5V: now also LED_R1.2, LED_R2.2
- net AGND: now also AGND1.2, LED1.C, LED2.C, R_VMTR_1.1, U$12.1
- net GND: no longer LED1.C
- net L: now also LEFTMOTOR.2; no longer LEFTMOTOR.1
- net LPWMA: now also LM.3; no longer LM.4
- net LPWMB: now also LM.4; no longer LM.3
- net MGND: now also AGND.1, AGND1.1, BAT.2, CB1.2, CB2.2, GND.1; no longer MGND.2
- net OUTA: now also U$17.OUT_B; no longer U$17.OUT_A
- net OUTB: now also U$17.OUT_A; no longer U$17.OUT_B
- net RPWMA: now also RM.2; no longer RM.1
- net RPWMB: now also RM.1; no longer RM.2
- net VBAT: now also R_VMTR_2.2
Other:
- moved on the sheet: CPWR_8
