File: Electrical Hardware/PCB 3rd version (Final Version)/peripheral/Peripherals.brd (EAGLE design)
At the start: 82 x 37 mm, 93 parts

Commit message: update PCB 3rd v
Parts:
- added LED2: BLUE, SparkFun-LED:LED-1206
- added LED_R2: 1k, SparkFun-Resistors:0805
- moved CC5 141.7 mm to (73.0, 63.0), turned to 0 degrees
- moved CC6 119.5 mm to (90.0, 56.0), turned to 270 degrees
- moved CC1 101.0 mm to (87.0, 55.0), turned to 0 degrees
- moved CC2 86.1 mm to (64.0, 56.0), turned to 90 degrees
- moved CRMC_1 85.0 mm to (104.0, 42.0)
- moved CPWR_9 82.3 mm to (86.0, 65.0), turned to 0 degrees
- moved LED_R1 81.0 mm to (72.0, 68.0)
- moved CPWR_7 75.2 mm to (82.0, 65.0)
- moved LED1 69.9 mm to (74.0, 70.0), turned to 0 degrees
- moved CPWR_3 67.1 mm to (81.0, 63.0)
- moved CPWR_2 64.1 mm to (72.0, 65.0), turned to 0 degrees
- moved CPWR_4 63.5 mm to (84.0, 55.0), turned to 270 degrees
- moved CPWR_8 60.9 mm to (67.0, 55.0)
- moved CPWR_1 59.2 mm to (73.0, 59.0), turned to 0 degrees
- moved CLMC_1 49.4 mm to (50.0, 42.0), turned to 0 degrees
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Connections:
- new net N$10: LED2.A, LED_R2.1
- net 3.3V: no longer LED_R1.2
- net A5V: now also LED_R1.2, LED_R2.2
- net AGND: now also LED1.C, LED2.C
- net GND: no longer LED1.C
Routing:
- net GND: track 24.9 -> 51.8 mm, vias 7 -> 12
- net VBAT: track 22.8 -> 44.0 mm, vias 2 -> 0
- net AGND: track 38.7 -> 58.1 mm, vias 27 -> 33
- net 5V: track 25.4 -> 44.3 mm, vias 4 -> 7
- net LENCA: track 7.11 -> 17.0 mm
- net MGND: track 29.4 -> 39.2 mm, vias 16 -> 18
- net 3.3V: track 7.44 -> 17.2 mm
- net RENCB: track 7.11 -> 16.1 mm
- net RENCA: track 11.5 -> 18.3 mm
- net LENCB: track 10.9 -> 17.5 mm
- net A5V: track 5.26 -> 10.9 mm, vias 0 -> 1
- net RE_LFB: track 9.76 -> 4.93 mm
- net RE_RFB: track 9.97 -> 6.32 mm
- net LPWMA: track 9.77 -> 7.29 mm
- net RPWMA: track 9.06 -> 6.64 mm
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Other:
- outline, holes or cut-outs redrawn
- board text added: "1st"
- board text added: "Eins"
- board text added: "The"
- board text added: "Triton"
- board text added: "UCSD"
- board text added: "~~~"

Commit message: Add safety guideline
Parts:
- LED_R1, LED_R2: value 1k -> 3k
- RRE1, RRE2, RRE3, RRE4: value 1.8k -> ~500ohm
- RRE5, RRE6: value 1.8k -> ~600ohm
Changed lines of the file:
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@@
 <attribute name="PROD_ID" value="RES-08474" x="-133" y="246" size="1.778" layer="27" display="off"/>
 </element>
-<element name="RRE1" library="SparkFun-Resistors" package="0805" value="1.8k" x="50" y="57">
+<element name="RRE1" library="SparkFun-Resistors" package="0805" value="~500ohm" x="50" y="57">
 <attribute name="PROD_ID" value="RES-08474" x="-116" y="237" size="1.778" layer="27" display="off"/>
 </element>
@@
 <attribute name="PROD_ID" value="RES-08474" x="228" y="263.99" size="1.778" layer="27" rot="R270" display="off"/>
 </element>
-<element name="RRE2" library="SparkFun-Resistors" package="0805" value="1.8k" x="54" y="68">
+<element name="RRE2" library="SparkFun-Resistors" package="0805" value="~500ohm" x="54" y="68">
 <attribute name="PROD_ID" value="RES-08474" x="-126" y="248" size="1.778" layer="27" display="off"/>
 </element>
@@
 <attribute name="PROD_ID" value="RES-08474" x="323" y="-119" size="1.778" layer="27" rot="R180" display="off"/>
 </element>
-<element name="RRE3" library="SparkFun-Resistors" package="0805" value="1.8k" x="99" y="70" rot="R180">
+<element name="RRE3" library="SparkFun-Resistors" package="0805" value="~500ohm" x="99" y="70" rot="R180">
 <attribute name="PROD_ID" value="RES-08474" x="299" y="-110" size="1.778" layer="27" rot="R180" display="off"/>
 </element>
@@
 <attribute name="PROD_ID" value="RES-08474" x="285" y="299" size="1.778" layer="27" rot="R270" display="off"/>
 </element>
-<element name="RRE4" library="SparkFun-Resistors" package="0805" value="1.8k" x="104" y="59" rot="R180">
+<element name="RRE4" library="SparkFun-Resistors" package="0805" value="~500ohm" x="104" y="59" rot="R180">
 <attribute name="PROD_ID" value="RES-08474" x="318" y="-121" size="1.778" layer="27" rot="R180" display="off"/>
 </element>
@@
 <attribute name="PROD_ID" value="RES-08474" x="228" y="304" size="1.778" layer="27" rot="R270" display="off"/>
 </element>
-<element name="RRE5" library="SparkFun-Resistors" package="0805" value="1.8k" x="39" y="44" rot="R270">
+<element name="RRE5" library="SparkFun-Resistors" package="0805" value="~600ohm" x="39" y="44" rot="R270">
 <attribute name="PROD_ID" value="RES-08474" x="219" y="278" size="1.778" layer="27" rot="R270" display="off"/>
 </element>
@@
 <attribute name="PROD_ID" value="RES-08474" x="286" y="334" size="1.778" layer="27" rot="R270" display="off"/>
 </element>
-<element name="RRE6" library="SparkFun-Resistors" package="0805" value="1.8k" x="112" y="46" rot="R270">
+<element name="RRE6" library="SparkFun-Resistors" package="0805" value="~600ohm" x="112" y="46" rot="R270">
 <attribute name="PROD_ID" value="RES-08474" x="292" y="306" size="1.778" layer="27" rot="R270" display="off"/>
 </element>
@@
 <attribute name="PROD_ID" value="CAP-08469" x="107" y="492" size="1.778" layer="27" rot="R270" display="off"/>
 </element>
-<element name="LED_R1" library="SparkFun-Resistors" package="0805" value="1k" x="72" y="68" rot="R180">
+<element name="LED_R1" library="SparkFun-Resistors" package="0805" value="3k" x="72" y="68" rot="R180">
 <attribute name="PROD_ID" value="RES-08474" x="687" y="58" size="1.778" layer="27" rot="R180" display="off"/>
 </element>
@@
 <attribute name="PROD_ID" value="RES-08474" x="112" y="39" size="1.778" layer="27" rot="R90" display="off"/>
 </element>
-<element name="LED_R2" library="SparkFun-Resistors" package="0805" value="1k" x="82" y="68">
+<element name="LED_R2" library="SparkFun-Resistors" package="0805" value="3k" x="82" y="68">
 <attribute name="PROD_ID" value="RES-08474" x="78" y="78" size="1.778" layer="27" display="off"/>
 </element>
