File: Electrical Hardware/PCB 3rd version (Final Version)/MCU/MCU.brd (EAGLE design)
At the start: 52 x 28 mm, 50 parts

Commit message: updated ADC
Parts:
- moved C2 2.27 mm to (62.3, 63.6), turned to 90 degrees
- moved C1 1.62 mm to (69.2, 63.5), turned to 90 degrees
- moved U$5 1.13 mm to (63.9, 61.9)
Routing:
- net OSC_OUT: track 9.91 -> 8.12 mm
Changed lines of the file:
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@@
 <attribute name="PROD_ID" value="CAP-08402" x="64.93" y="18.9" size="1.778" layer="27" rot="R90" display="off"/>
 </element>
-<element name="C1" library="SparkFun-Capacitors" package="0603" value="12pF" x="69.48" y="65.13">
-<attribute name="PROD_ID" value="CAP-07876" x="17.48" y="87.13" size="1.778" layer="27" display="off"/>
-</element>
-<element name="C2" library="SparkFun-Capacitors" package="0603" value="12pF" x="63.98" y="65.12" rot="R180">
-<attribute name="PROD_ID" value="CAP-07876" x="121.98" y="47.12" size="1.778" layer="27" rot="R180" display="off"/>
-</element>
-<element name="U$5" library="Cristal Oscillator" package="OSC" value="OSC" x="64.83" y="62.5"/>
+<element name="C1" library="SparkFun-Capacitors" package="0603" value="12pF" x="69.21" y="63.53" rot="R90">
+<attribute name="PROD_ID" value="CAP-07876" x="47.21" y="11.53" size="1.778" layer="27" rot="R90" display="off"/>
+</element>
+<element name="C2" library="SparkFun-Capacitors" package="0603" value="12pF" x="62.32" y="63.57" rot="R90">
+<attribute name="PROD_ID" value="CAP-07876" x="44.32" y="5.57" size="1.778" layer="27" rot="R90" display="off"/>
+</element>
+<element name="U$5" library="Cristal Oscillator" package="OSC" value="OSC" x="63.86" y="61.92"/>
 <element name="LM1" library="headers(2mm)" package="1X4" value="1X4" x="90" y="70"/>
 <element name="CH4" library="SparkFun-Resistors" package="0805" value="22ohm" x="62" y="48">
@@
 <wire x1="82.79" y1="66.91" x2="82.8" y2="66.92" width="0.3048" layer="1"/>
 <via x="82.8" y="66.92" extent="1-16" drill="0.35"/>
-<wire x1="63.13" y1="65.12" x2="63.09" y2="65.08" width="0.3048" layer="1"/>
-<wire x1="63.09" y1="65.08" x2="61.93" y2="65.08" width="0.3048" layer="1"/>
-<via x="61.93" y="65.08" extent="1-16" drill="0.35"/>
-<wire x1="70.33" y1="65.13" x2="70.33" y2="63.87" width="0.3048" layer="1"/>
-<wire x1="70.33" y1="63.87" x2="70.34" y2="63.86" width="0.3048" layer="1"/>
-<via x="70.34" y="63.86" extent="1-16" drill="0.35"/>
 <wire x1="68.79" y1="67.13" x2="68.76" y2="67.16" width="0.3048" layer="1"/>
 <wire x1="68.76" y1="67.16" x2="67.77" y2="67.16" width="0.3048" layer="1"/>
@@
 <contactref element="LED2" pad="C"/>
 <contactref element="LED4" pad="C"/>
+<wire x1="62.32" y1="64.42" x2="63.67" y2="64.42" width="0.3048" layer="1"/>
+<wire x1="63.67" y1="64.42" x2="63.69" y2="64.44" width="0.3048" layer="1"/>
+<via x="63.69" y="64.44" extent="1-16" drill="0.35"/>
+<wire x1="69.21" y1="64.38" x2="67.73" y2="64.38" width="0.3048" layer="1"/>
+<wire x1="67.73" y1="64.38" x2="67.67" y2="64.44" width="0.3048" layer="1"/>
+<via x="67.67" y="64.44" extent="1-16" drill="0.35"/>
 <wire x1="3.63" y1="-2.41" x2="8.34" y2="-2.41" width="0" layer="19" extent="1-1"/>
 <wire x1="3.63" y1="-7.08" x2="3.63" y2="-2.41" width="0" layer="19" extent="1-1"/>
@@
 <contactref element="C1" pad="1"/>
 <contactref element="U$5" pad="P$2"/>
-<wire x1="71.25" y1="60.75" x2="70.13" y2="60.75" width="0.3048" layer="1"/>
-<wire x1="70.13" y1="60.75" x2="68.63" y2="62.25" width="0.3048" layer="1"/>
-<wire x1="68.63" y1="62.25" x2="68.63" y2="62.6" width="0.3048" layer="1"/>
-<wire x1="68.63" y1="62.6" x2="68.63" y2="65.13" width="0.3048" layer="1"/>
+<wire x1="69.21" y1="62.68" x2="68.32" y2="62.68" width="0.3048" layer="1"/>
+<wire x1="68.32" y1="62.68" x2="67.71" y2="62.07" width="0.3048" layer="1"/>
+<wire x1="67.71" y1="62.07" x2="67.66" y2="62.02" width="0.3048" layer="1"/>
+<wire x1="71.25" y1="60.75" x2="69.03" y2="60.75" width="0.3048" layer="1"/>
+<wire x1="69.03" y1="60.75" x2="67.71" y2="62.07" width="0.3048" layer="1"/>
 </signal>
 <signal name="OSC_OUT">
@@
 <contactref element="C2" pad="1"/>
 <contactref element="U$5" pad="P$1"/>
-<wire x1="71.25" y1="60.25" x2="69.86" y2="60.25" width="0.3048" layer="1"/>
-<wire x1="66.39" y1="61.04" x2="64.83" y2="62.6" width="0.3048" layer="1"/>
-<wire x1="69.86" y1="60.25" x2="69.07" y2="61.04" width="0.3048" layer="1"/>
-<wire x1="69.07" y1="61.04" x2="66.39" y2="61.04" width="0.3048" layer="1"/>
-<wire x1="64.83" y1="62.6" x2="64.83" y2="65.12" width="0.3048" layer="1"/>
+<wire x1="71.25" y1="60.25" x2="65.63" y2="60.25" width="0.3048" layer="1"/>
+<wire x1="65.63" y1="60.25" x2="63.86" y2="62.02" width="0.3048" layer="1"/>
+<wire x1="63.86" y1="62.02" x2="62.32" y2="62.72" width="0" layer="19" extent="1-1"/>
 </signal>
 <signal name="VCAP_1">

Commit message: finalized PCB
Parts:
- removed LED4: BLUE, SparkFun-LED:LED-1206
- removed LED_R4: 1k, SparkFun-Resistors:0805
- added BUTTON: 1X2, headers(2mm):1X2
- added RSTC: 0.1uf, SparkFun-Capacitors:0805
- added RSTR: 47K, SparkFun-Resistors:0805
- moved LED1 115.4 mm to (93.6, 68.0)
- moved LED_R1 111.8 mm to (91.2, 66.0), turned to 180 degrees
- moved LED_R2 98.8 mm to (62.8, 66.1)
- moved LED2 88.5 mm to (60.4, 68.0), turned to 180 degrees
Connections:
- removed net LED3: LED_R4.2, U$4.PC12
- removed net N$15: LED4.A, LED_R4.1
- net 3.3V: now also RSTR.2
- net GND: now also BUTTON.1, RSTC.2; no longer LED4.C
- net LED2: now also U$4.PC15; no longer U$4.PC11
- net RESET: now also BUTTON.2, RSTC.1, RSTR.1
Routing:
- net LED1: track 0.00 -> 13.6 mm
- net LED2: track 0.00 -> 11.4 mm, vias 0 -> 2
- net RESET: track 31.4 -> 39.9 mm
- net 3.3V: track 16.0 -> 24.2 mm, vias 0 -> 1
- net GND: track 18.9 -> 23.8 mm, vias 14 -> 17
- net N$14: track 0.00 -> 1.96 mm
- net N$13: track 0.00 -> 1.87 mm
- net OSC_OUT: track 8.12 -> 9.95 mm
Other:
- board size 52 x 28 mm -> 40 x 28 mm

Commit message: minor updates
Parts:
- B1: value 1k -> 47k
Changed lines of the file:
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@@
 <attribute name="PROD_ID" value="RES-08474" x="92" y="50" size="1.778" layer="27" display="off"/>
 </element>
-<element name="B1" library="SparkFun-Resistors" package="0805" value="1k" x="85.75" y="50.64" rot="R180">
+<element name="B1" library="SparkFun-Resistors" package="0805" value="47k" x="85.75" y="50.64" rot="R180">
 <attribute name="PROD_ID" value="RES-08474" x="85.75" y="50.64" size="1.778" layer="27" rot="R180" display="off"/>
 </element>
