File: Electrical Hardware/PCB 3rd version (Final Version)/MCU/MCU.sch (EAGLE design)
At the start: 50 parts

Commit message: finalized PCB
Parts:
- removed LED4: BLUE, SparkFun-LED:LED-BLUE1206
- removed LED_R4: 1k, SparkFun-Resistors:0.75OHM-0805-1/4W-1%
- added BUTTON: 1X2, headers(2mm):1X2
- added RSTC: 0.1uf, SparkFun-Capacitors:22UF-0805-6.3V-20%
- added RSTR: 47K, SparkFun-Resistors:0.75OHM-0805-1/4W-1%
Connections:
- removed net LED3: LED_R4.2, U$4.PC12
- removed net N$15: LED4.A, LED_R4.1
- net 3.3V: now also RSTR.2
- net GND: now also BUTTON.1, RSTC.2; no longer LED4.C
- net LED2: now also U$4.PC15; no longer U$4.PC11
- net RESET: now also BUTTON.2, RSTC.1, RSTR.1
Changed lines of the file:
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@@
 <part name="LED_R1" library="SparkFun-Resistors" deviceset="0.75OHM" device="-0805-1/4W-1%" value="1k"/>
 <part name="LED1" library="SparkFun-LED" deviceset="LED-BLUE" device="1206" value="BLUE"/>
-<part name="LED_R4" library="SparkFun-Resistors" deviceset="0.75OHM" device="-0805-1/4W-1%" value="1k"/>
-<part name="LED4" library="SparkFun-LED" deviceset="LED-BLUE" device="1206" value="BLUE"/>
+<part name="RSTR" library="SparkFun-Resistors" deviceset="0.75OHM" device="-0805-1/4W-1%" value="47K"/>
+<part name="RSTC" library="SparkFun-Capacitors" deviceset="22UF" device="-0805-6.3V-20%" value="0.1uf"/>
+<part name="GND7" library="supply1" library_urn="urn:adsk.eagle:library:371" deviceset="GND" device=""/>
+<part name="BUTTON" library="headers(2mm)" deviceset="1X2" device=""/>
 </parts>
 <sheets>
@@
 <instance part="LED_R1" gate="G$1" x="10.16" y="99.06" rot="R270"/>
 <instance part="LED1" gate="G$1" x="10.16" y="114.3" rot="R180"/>
-<instance part="LED_R4" gate="G$1" x="33.02" y="99.06" rot="R270"/>
-<instance part="LED4" gate="G$1" x="33.02" y="114.3" rot="R180"/>
+<instance part="RSTR" gate="G$1" x="114.3" y="73.66" rot="R180"/>
+<instance part="RSTC" gate="G$1" x="124.46" y="66.04"/>
+<instance part="GND7" gate="1" x="129.54" y="55.88"/>
+<instance part="BUTTON" gate="G$1" x="139.7" y="50.8" rot="R90"/>
 </instances>
 <busses>
@@
 </segment>
 <segment>
-<pinref part="LED4" gate="G$1" pin="C"/>
-<wire x1="33.02" y1="119.38" x2="33.02" y2="124.46" width="0.1524" layer="91"/>
-<label x="33.02" y="124.46" size="0.8128" layer="95" rot="R90" xref="yes"/>
+<pinref part="GND7" gate="1" pin="GND"/>
+<wire x1="129.54" y1="58.42" x2="129.54" y2="63.5" width="0.1524" layer="91"/>
+<pinref part="RSTC" gate="G$1" pin="2"/>
+<wire x1="129.54" y1="63.5" x2="124.46" y2="63.5" width="0.1524" layer="91"/>
+<wire x1="129.54" y1="63.5" x2="139.7" y2="63.5" width="0.1524" layer="91"/>
+<junction x="129.54" y="63.5"/>
+<pinref part="BUTTON" gate="G$1" pin="1"/>
+<wire x1="139.7" y1="63.5" x2="139.7" y2="53.34" width="0.1524" layer="91"/>
 </segment>
 </net>
@@
 <wire x1="-119.38" y1="-55.88" x2="-119.38" y2="-48.26" width="0.1524" layer="91"/>
 </segment>
+<segment>
+<wire x1="106.68" y1="73.66" x2="109.22" y2="73.66" width="0.1524" layer="91"/>
+<label x="106.68" y="73.66" size="0.8128" layer="95" rot="R180" xref="yes"/>
+<pinref part="RSTR" gate="G$1" pin="2"/>
+</segment>
 </net>
 <net name="EM_RF" class="0">
@@
 <wire x1="-76.2" y1="-55.88" x2="-76.2" y2="-50.8" width="0.1524" layer="91"/>
 </segment>
+<segment>
+<pinref part="RSTR" gate="G$1" pin="1"/>
+<wire x1="119.38" y1="73.66" x2="124.46" y2="73.66" width="0.1524" layer="91"/>
+<label x="139.7" y="73.66" size="0.8128" layer="95" xref="yes"/>
+<pinref part="RSTC" gate="G$1" pin="1"/>
+<wire x1="124.46" y1="73.66" x2="134.62" y2="73.66" width="0.1524" layer="91"/>
+<wire x1="134.62" y1="73.66" x2="139.7" y2="73.66" width="0.1524" layer="91"/>
+<wire x1="124.46" y1="71.12" x2="124.46" y2="73.66" width="0.1524" layer="91"/>
+<junction x="124.46" y="73.66"/>
+<wire x1="144.78" y1="68.58" x2="134.62" y2="68.58" width="0.1524" layer="91"/>
+<wire x1="134.62" y1="68.58" x2="134.62" y2="73.66" width="0.1524" layer="91"/>
+<junction x="134.62" y="73.66"/>
+<wire x1="144.78" y1="68.58" x2="144.78" y2="55.88" width="0.1524" layer="91"/>
+<wire x1="144.78" y1="55.88" x2="142.24" y2="55.88" width="0.1524" layer="91"/>
+<pinref part="BUTTON" gate="G$1" pin="2"/>
+<wire x1="142.24" y1="55.88" x2="142.24" y2="53.34" width="0.1524" layer="91"/>
+</segment>
 </net>
 <net name="OSC_IN" class="0">
@@
 </segment>
 </net>
-<net name="N$15" class="0">
-<segment>
-<pinref part="LED_R4" gate="G$1" pin="1"/>
-<pinref part="LED4" gate="G$1" pin="A"/>
-<wire x1="33.02" y1="111.76" x2="33.02" y2="104.14" width="0.1524" layer="91"/>
-</segment>
-</net>
 <net name="LED1" class="0">
 <segment>
@@
 </segment>
 <segment>
-<pinref part="U$4" gate="G$1" pin="PC11"/>
-<wire x1="12.7" y1="38.1" x2="12.7" y2="40.64" width="0.1524" layer="91"/>
-<label x="12.7" y="40.64" size="0.8128" layer="95" rot="R90" xref="yes"/>
-</segment>
-</net>
-<net name="LED3" class="0">
-<segment>
-<pinref part="LED_R4" gate="G$1" pin="2"/>
-<wire x1="33.02" y1="93.98" x2="33.02" y2="91.44" width="0.1524" layer="91"/>
-<label x="33.02" y="91.44" size="0.8128" layer="95" rot="R270" xref="yes"/>
-</segment>
-<segment>
-<pinref part="U$4" gate="G$1" pin="PC12"/>
-<wire x1="10.16" y1="38.1" x2="10.16" y2="40.64" width="0.1524" layer="91"/>
-<label x="10.16" y="40.64" size="0.8128" layer="95" rot="R90" xref="yes"/>
-</segment>
-</net>
+<label x="-43.18" y="12.7" size="0.8128" layer="95" rot="R180" xref="yes"/>
+<pinref part="U$4" gate="G$1" pin="PC15"/>
+<wire x1="-43.18" y1="12.7" x2="-35.56" y2="12.7" width="0.1524" layer="91"/>
+</segment>
+</net>

Commit message: minor updates
Parts:
- B1: value 1k -> 47k
Changed lines of the file:
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@@
 <part name="CH7" library="SparkFun-Resistors" deviceset="0.75OHM" device="-0805-1/4W-1%" value="22ohm"/>
 <part name="CH8" library="SparkFun-Resistors" deviceset="0.75OHM" device="-0805-1/4W-1%" value="22ohm"/>
-<part name="B1" library="SparkFun-Resistors" deviceset="0.75OHM" device="-0805-1/4W-1%" value="1k"/>
+<part name="B1" library="SparkFun-Resistors" deviceset="0.75OHM" device="-0805-1/4W-1%" value="47k"/>
 <part name="CH9" library="SparkFun-Resistors" deviceset="0.75OHM" device="-0805-1/4W-1%" value="22ohm"/>
 <part name="CH10" library="SparkFun-Resistors" deviceset="0.75OHM" device="-0805-1/4W-1%" value="22ohm"/>
